Commit message: 1
1

File: ocs2_pros_gazebo2/urdf/pros_walker.urdf (robot description, URDF)
Before this commit: robot pros_walker, 17 links, 16 joints
Links:
- added link fp1_l, mass 0.1; collision sphere radius=0.01; collision sphere radius=0.01
- added link fp1_r, mass 0.1; collision sphere radius=0.01; collision sphere radius=0.01
- added link fp2_l, mass 0.1; collision sphere radius=0.01; collision sphere radius=0.01
- added link fp2_r, mass 0.1; collision sphere radius=0.01; collision sphere radius=0.01
- added link fp3_l, mass 0.1; collision sphere radius=0.01; collision sphere radius=0.01
- added link fp3_r, mass 0.1; collision sphere radius=0.01; collision sphere radius=0.01
- added link fp4_l, mass 0.1; collision sphere radius=0.01; collision sphere radius=0.01
- added link fp4_r, mass 0.1; collision sphere radius=0.01; collision sphere radius=0.01
Joints:
- added joint fp1_fixed_l_foot: type fixed, parent l_foot, child fp1_l, origin xyz=0.18 0.03 -0.08 rpy=0 0 0
- added joint fp1_fixed_r_foot: type fixed, parent r_foot, child fp1_r, origin xyz=0.18 0.03 -0.08 rpy=0 0 0
- added joint fp2_fixed_l_foot: type fixed, parent l_foot, child fp2_l, origin xyz=0.18 -0.03 -0.08 rpy=0 0 0
- added joint fp2_fixed_r_foot: type fixed, parent r_foot, child fp2_r, origin xyz=0.18 -0.03 -0.08 rpy=0 0 0
- added joint fp3_fixed_l_foot: type fixed, parent l_foot, child fp3_l, origin xyz=-0.08 0.035 -0.08 rpy=0 0 0
- added joint fp3_fixed_r_foot: type fixed, parent r_foot, child fp3_r, origin xyz=-0.08 0.035 -0.08 rpy=0 0 0
- added joint fp4_fixed_l_foot: type fixed, parent l_foot, child fp4_l, origin xyz=-0.08 -0.035 -0.08 rpy=0 0 0
- added joint fp4_fixed_r_foot: type fixed, parent r_foot, child fp4_r, origin xyz=-0.08 -0.035 -0.08 rpy=0 0 0

Commit message: 1
1

File: ocs2_pros_gazebo2/urdf/pros_walker.urdf (robot description, URDF)
Before this commit: robot pros_walker, 25 links, 24 joints
Links:
- removed link pelvis
- removed link pelvis_inertia
- added link base; collision box size=0.1 0.15 0.2; collision cylinder length=0.05 radius=0.16
- added link base_inertia, mass 14.2529
Joints:
- removed joint pelvis_to_pelvis_inertia
- added joint base_to_base_inertia: type fixed, parent base, child base_inertia, origin xyz=0 0 0 rpy=0 0 0
- joint back_lbz: parent pelvis -> base
- joint l_leg_uhz: parent pelvis -> base
- joint r_leg_uhz: parent pelvis -> base

Commit message: 1

File: ocs2_pros_gazebo2/urdf/pros_walker.urdf (robot description, URDF)
Before this commit: robot pros_walker, 25 links, 24 joints
Links:
- removed link ltorso
- removed link mtorso
- removed link utorso
- added link fp0_l, mass 0.1; collision sphere radius=0.01; collision sphere radius=0.01
- added link fp0_r, mass 0.1; collision sphere radius=0.01; collision sphere radius=0.01
Joints:
- removed joint back_lbz
- removed joint back_mby
- removed joint back_ubx
- added joint fp0_fixed_l_foot: type fixed, parent l_foot, child fp0_l, origin xyz=0.05 0 -0.08 rpy=0 0 0
- added joint fp0_fixed_r_foot: type fixed, parent r_foot, child fp0_r, origin xyz=0.05 0 -0.08 rpy=0 0 0
